File: PCB/BUTTON SMASHER, NOISE MAKER1.kicad_pcb (KiCad board)
At the start: 2 copper layers, 95.4 x 95.4 mm, 13 parts, among them SW1 SW_Push, SW2 SW_Push, SW3 SW_Push, U1 XIAO-RP2040-DIP

Commit message: Add files via upload
Other:
- board text added: "BEEP BEEP BEEP"
- board text added: "MUSIC PLAYER"

Commit message: Add files via upload
Other:
- outline, holes or cut-outs redrawn

Commit message: Add files via upload
Parts:
- moved D1 31.2 mm to (120.5, 132.0)
- moved BZ1 11.1 mm to (127.4, 126.5)
- moved R1 8.73 mm to (118.5, 93.0)
Routing:
- net Net-(D1-PadA): track 8.47 -> 66.7 mm, vias 0 -> 1
- net GND: track 234.6 -> 254.1 mm
- net Net-(U1-P29_A3_D3): track 27.8 -> 19.0 mm
- net Net-(BZ1-+): track 19.8 -> 25.9 mm
Changed lines of the file:
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@@
 			(drillshape 0)
 			(scaleselection 1)
-			(outputdirectory "../gerber and drill/")
+			(outputdirectory "gerber and drill/")
 		)
 	)
 	(footprint "footprints:LEDRD254W57D500H1070"
 		(layer "F.Cu")
-		(at 129.23 102)
+		(at 120.5 132)
 		(property "Reference" "D1"
 			(at 0.04 -3.708 0)
@@
 	(footprint "Resistor_THT:R_Axial_DIN0204_L3.6mm_D1.6mm_P5.08mm_Horizontal"
 		(layer "F.Cu")
-		(at 126.96 95)
+		(at 118.46 93)
 		(descr "Resistor, Axial_DIN0204 series, Axial, Horizontal, pin pitch=5.08mm, 0.167W, length*diameter=3.6*1.6mm^2, http://cdn-reichelt.de/documents/datenblatt/B400/1_4W%23YAG.pdf")
 		(tags "Resistor Axial_DIN0204 series Axial Horizontal pin pitch 5.08mm 0.167W length 3.6mm diameter 1.6mm")
@@
 	(footprint "Buzzer_Beeper:Buzzer_12x9.5RM7.6"
 		(layer "F.Cu")
-		(at 126.2 115.5)
+		(at 127.4 126.5)
 		(descr "Generic Buzzer, D12mm height 9.5mm with RM7.6mm")
 		(tags "buzzer")
@@
 	)
 	(segment
-		(start 126.96 98.46)
-		(end 130.5 102)
+		(start 118.04 117.585786)
+		(end 118.625786 117)
 		(width 0.2)
 		(layer "F.Cu")
@@
 	)
 	(segment
-		(start 126.96 95)
-		(end 126.96 98.46)
+		(start 130.74 102.74)
+		(end 134.7 102.74)
 		(width 0.2)
 		(layer "F.Cu")
@@
 	)
 	(segment
+		(start 118.625786 117)
+		(end 133.572792 117)
+		(width 0.2)
+		(layer "F.Cu")
+		(net "Net-(D1-PadA)")
+	)
+	(segment
+		(start 125 97)
+		(end 130.74 102.74)
+		(width 0.2)
+		(layer "F.Cu")
+		(net "Net-(D1-PadA)")
+	)
+	(segment
+		(start 134.7 115.872792)
+		(end 134.7 102.74)
+		(width 0.2)
+		(layer "F.Cu")
+		(net "Net-(D1-PadA)")
+	)
+	(segment
+		(start 121.77 132)
+		(end 121.77 122.144214)
+		(width 0.2)
+		(layer "F.Cu")
+		(net "Net-(D1-PadA)")
+	)
+	(segment
+		(start 133.572792 117)
+		(end 134.7 115.872792)
+		(width 0.2)
+		(layer "F.Cu")
+		(net "Net-(D1-PadA)")
+	)
+	(segment
+		(start 121.77 122.144214)
+		(end 118.04 118.414214)
+		(width 0.2)
+		(layer "F.Cu")
+		(net "Net-(D1-PadA)")
+	)
+	(segment
+		(start 118.04 118.414214)
+		(end 118.04 117.585786)
+		(width 0.2)
+		(layer "F.Cu")
+		(net "Net-(D1-PadA)")
+	)
+	(via
+		(at 125 97)
+		(size 0.6)
+		(drill 0.3)
+		(layers "F.Cu" "B.Cu")
+		(net "Net-(D1-PadA)")
+	)
+	(segment
+		(start 122.46 97)
+		(end 125 97)
+		(width 0.2)
+		(layer "B.Cu")
+		(net "Net-(D1-PadA)")
+	)
+	(segment
+		(start 118.46 93)
+		(end 122.46 97)
+		(width 0.2)
+		(layer "B.Cu")
+		(net "Net-(D1-PadA)")
+	)
+	(segment
 		(start 104.11 79.46)
 		(end 100.17 75.52)
@@
 	)
 	(segment
+		(start 128.2925 133.2075)
+		(end 120.4375 133.2075)
+		(width 0.2)
+		(layer "F.Cu")
+		(net "GND")
+	)
+	(segment
 		(start 90.380101 78.32)
 		(end 91.539899 78.32)
@@
 	)
 	(segment
+		(start 114.96 127.73)
+		(end 119.23 132)
+		(width 0.2)
+		(layer "F.Cu")
+		(net "GND")
+	)
+	(segment
 		(start 90.3 116.5)
 		(end 95.242 111.558)
@@
 	)
 	(segment
+		(start 114.96 125)
+		(end 114.96 127.73)
+		(width 0.2)
+		(layer "F.Cu")
+		(net "GND")
+	)
+	(segment
 		(start 103.6295 97.819895)
 		(end 107.809605 102)
@@
 	)
 	(segment
+		(start 120.4375 133.2075)
+		(end 119.23 132)
+		(width 0.2)
+		(layer "F.Cu")
+		(net "GND")
+	)
+	(segment
 		(start 105.8 126.5)
 		(end 105.8 112.549605)
@@
 	)
 	(segment
-		(start 127.96 109.66)
-		(end 133.8 115.5)
+		(start 135 126.5)
+		(end 128.2925 133.2075)
 		(width 0.2)
 		(layer "F.Cu")
@@
 	)
 	(segment
-		(start 108.2935 98.442)
-		(end 107.2315 97.38)
+		(start 120.733395 93)
+		(end 115.291395 98.442)
 		(width 0.2)
 		(layer "F.Cu")
@@
 	)
 	(segment
-		(start 130.64 93.6)
-		(end 120.133395 93.6)
+		(start 108.2935 98.442)
+		(end 107.2315 97.38)
 		(width 0.2)
 		(layer "F.Cu")
@@
 	)
 	(segment
-		(start 132.04 95)
-		(end 130.64 93.6)
+		(start 123.54 93)
+		(end 120.733395 93)
 		(width 0.2)
 		(layer "F.Cu")
@@
 	)
 	(segment
-		(start 120.133395 93.6)
-		(end 115.291395 98.442)
+		(start 123.874214 126.5)
+		(end 111.056214 113.682)
 		(width 0.2)
-		(layer "F.Cu")
-		(net "Net-(U1-P29_A3_D3)")
+		(layer "B.Cu")
+		(net "Net-(BZ1-+)")
 	)
 	(segment
-		(start 126.2 115.5)
-		(end 109.2765 115.5)
+		(start 111.056214 113.682)
+		(end 108.2935 113.682)
 		(width 0.2)
-		(layer "F.Cu")
+		(layer "B.Cu")
 		(net "Net-(BZ1-+)")
 	)
 	(segment
-		(start 109.2765 115.5)
-		(end 107.2315 113.455)
+		(start 127.4 126.5)
+		(end 123.874214 126.5)
 		(width 0.2)
-		(layer "F.Cu")
+		(layer "B.Cu")
+		(net "Net-(BZ1-+)")
+	)
+	(segment
+		(start 108.2935 113.682)
+		(end 107.2315 112.62)
+		(width 0.2)
+		(layer "B.Cu")
 		(net "Net-(BZ1-+)")
 	)
@@
 	)
 	(segment
-		(start 135.1 101.725786)
-		(end 135.1 116.038478)
+		(start 126.522893 94.022893)
+		(end 134.225786 101.725786)
 		(width 0.2)
 		(layer "F.Cu")
@@
 	)
 	(segment
-		(start 127.374214 94)
+		(start 134.225786 101.725786)
 		(end 135.1 101.725786)
 		(width 0.2)
@@
 	)
 	(segment
-		(start 121.354286 99.1915)
-		(end 126.545786 94)
+		(start 135.1 101.725786)
+		(end 135.1 116.038478)
 		(width 0.2)
 		(layer "F.Cu")
@@
 	)
 	(segment
-		(start 126.545786 94)
-		(end 127.374214 94)
+		(start 121.354286 99.1915)
+		(end 126.522893 94.022893)
 		(width 0.2)
 		(layer "F.Cu")
