File: BUTTON SMASHER, NOISE MAKER1.kicad_pcb (KiCad board)
At the start: 2 copper layers, 95.4 x 95.4 mm, 13 parts, among them SW1 SW_Push, SW2 SW_Push, SW3 SW_Push, U1 XIAO-RP2040-DIP

Commit message: Add files via upload
Parts:
- moved U1 32.2 mm to (133.2, 124.0)
- moved D1 26.0 mm to (121.5, 106.0)
- moved BZ1 24.1 mm to (129.9, 102.5)
- moved D2 6.94 mm to (112.0, 130.5)
- moved R2 6.08 mm to (108.0, 119.0)
Routing:
- net Net-(U1-P27_A1_D1): track 20.4 -> 102.5 mm
- net Net-(U1-P28_A2_D2): track 27.4 -> 83.6 mm
- net Net-(U1-P6_SDA_D4): track 67.7 -> 18.7 mm
- net Net-(D1-PadA): track 66.7 -> 19.2 mm
- net Net-(U1-P26_A0_D0): track 26.4 -> 69.4 mm
- net Net-(U1-P7_SCL_D5): track 14.1 -> 49.9 mm
- net Net-(BZ2-+): track 15.7 -> 51.1 mm
- net Net-(BZ3-+): track 21.8 -> 55.6 mm
- net Net-(U1-P29_A3_D3): track 19.0 -> 36.0 mm
- net Net-(BZ1-+): track 25.9 -> 40.3 mm
- net GND: track 254.1 -> 241.4 mm
- net Net-(D2-PadA): track 8.47 -> 13.7 mm
